File: power.sch (KiCad schematic (older format))
At the start: 9 parts, among them CON1 BARREL_JACK, U2 AP3211

Commit message: ksch: use schottky diode for switching regulator
Parts:
- removed D1: Diode, symbol D_Small_ALT
- added D1: D_Schottky_Small_ALT, symbol D_Schottky_Small_ALT
Connections:
- wire segments 14 -> 17
Changed lines of the file:
@@
 LIBS:valves
 LIBS:openloop
-LIBS:looper-cache
 EELAYER 25 0
 EELAYER END
@@
 $EndComp
 $Comp
-L GND #PWR01
+L GND #PWR1
 U 1 1 58B351BB
 P 2450 1750
-F 0 "#PWR01" H 2450 1500 50  0001 C CNN
+F 0 "#PWR1" H 2450 1500 50  0001 C CNN
 F 1 "GND" H 2450 1600 50  0000 C CNN
 F 2 "" H 2450 1750 50  0000 C CNN
@@
 9V
 $Comp
-L PWR_FLAG #FLG02
+L PWR_FLAG #FLG1
 U 1 1 58B352C2
 P 1950 1550
-F 0 "#FLG02" H 1950 1645 50  0001 C CNN
+F 0 "#FLG1" H 1950 1645 50  0001 C CNN
 F 1 "PWR_FLAG" H 1950 1730 50  0000 C CNN
 F 2 "" H 1950 1550 50  0000 C CNN
@@
 $EndComp
 $Comp
-L PWR_FLAG #FLG03
+L PWR_FLAG #FLG2
 U 1 1 58B35302
 P 1950 1750
-F 0 "#FLG03" H 1950 1845 50  0001 C CNN
+F 0 "#FLG2" H 1950 1845 50  0001 C CNN
 F 1 "PWR_FLAG" H 1950 1930 50  0000 C CNN
 F 2 "" H 1950 1750 50  0000 C CNN
@@
 Wire Wire Line
 	4500 1550 4600 1550
-$Comp
-L D_Small_ALT D1
-U 1 1 58B356A7
-P 4750 1850
-F 0 "D1" H 4700 1930 50  0000 L CNN
-F 1 "Diode" H 4650 1800 50  0001 L CNN
-F 2 "" V 4750 1850 50  0000 C CNN
-F 3 "" V 4750 1850 50  0000 C CNN
-	1    4750 1850
-	0    1    1    0
-$EndComp
 $Comp
 L L_Small L1
@@
 L R_Small R1
 U 1 1 58B360A5
-P 5250 1850
-F 0 "R1" H 5280 1870 50  0000 L CNN
-F 1 "68k" H 5280 1810 50  0000 L CNN
-F 2 "" H 5250 1850 50  0000 C CNN
-F 3 "" H 5250 1850 50  0000 C CNN
-	1    5250 1850
+P 6050 1850
+F 0 "R1" H 6080 1870 50  0000 L CNN
+F 1 "68k" H 6080 1810 50  0000 L CNN
+F 2 "" H 6050 1850 50  0000 C CNN
+F 3 "" H 6050 1850 50  0000 C CNN
+	1    6050 1850
 	1    0    0    -1
 $EndComp
@@
 L R_Small R2
 U 1 1 58B360E7
-P 5250 2150
-F 0 "R2" H 5280 2170 50  0000 L CNN
-F 1 "12k" H 5280 2110 50  0000 L CNN
-F 2 "" H 5250 2150 50  0000 C CNN
-F 3 "" H 5250 2150 50  0000 C CNN
-	1    5250 2150
+P 6050 2150
+F 0 "R2" H 6080 2170 50  0000 L CNN
+F 1 "12k" H 6080 2110 50  0000 L CNN
+F 2 "" H 6050 2150 50  0000 C CNN
+F 3 "" H 6050 2150 50  0000 C CNN
+	1    6050 2150
 	1    0    0    -1
 $EndComp
@@
 L C_Small C3
 U 1 1 58B3611B
-P 5750 1850
-F 0 "C3" H 5760 1920 50  0000 L CNN
-F 1 "22uF" H 5850 1850 50  0000 L CNN
-F 2 "" H 5750 1850 50  0000 C CNN
-F 3 "" H 5750 1850 50  0000 C CNN
-	1    5750 1850
-	1    0    0    -1
-$EndComp
-$Comp
-L GND #PWR04
+P 5300 1850
+F 0 "C3" H 5310 1920 50  0000 L CNN
+F 1 "22uF" H 5400 1850 50  0000 L CNN
+F 2 "" H 5300 1850 50  0000 C CNN
+F 3 "" H 5300 1850 50  0000 C CNN
+	1    5300 1850
+	1    0    0    -1
+$EndComp
+$Comp
+L GND #PWR2
 U 1 1 58B36556
 P 4750 2250
-F 0 "#PWR04" H 4750 2000 50  0001 C CNN
+F 0 "#PWR2" H 4750 2000 50  0001 C CNN
 F 1 "GND" H 4750 2100 50  0000 C CNN
 F 2 "" H 4750 2250 50  0000 C CNN
@@
 Wire Wire Line
 	5150 1750 6150 1750
-Connection ~ 5250 1750
-Wire Wire Line
-	5750 2250 5750 1950
-Wire Wire Line
-	4750 2250 5750 2250
-Connection ~ 5250 2250
+Connection ~ 6050 1750
+Connection ~ 6050 2250
 Wire Wire Line
 	4750 1950 4750 2250
 Wire Wire Line
-	5250 1950 4500 1950
-Wire Wire Line
-	5250 1950 5250 2050
-Connection ~ 5250 1950
+	6050 1950 6050 2050
+Connection ~ 6050 1950
 Connection ~ 3550 1750
 Connection ~ 3650 1550
-Connection ~ 5750 1750
+Connection ~ 5300 1750
 Text Label 6150 1750 0    60   ~ 0
 5.4V
+Wire Wire Line
+	4750 2250 6050 2250
+Wire Wire Line
+	5300 1950 5300 2250
+Connection ~ 5300 2250
+Wire Wire Line
+	6050 1950 6200 1950
+Wire Wire Line
+	6200 1950 6200 2400
+Wire Wire Line
+	6200 2400 4500 2400
+Wire Wire Line
+	4500 2400 4500 1950
+$Comp
+L D_Schottky_Small_ALT D1
+U 1 1 58B38399
+P 4750 1850
+F 0 "D1" H 4700 1930 50  0000 L CNN
+F 1 "D_Schottky_Small_ALT" H 4470 1770 50  0001 L CNN
+F 2 "" V 4750 1850 50  0000 C CNN
+F 3 "" V 4750 1850 50  0000 C CNN
+	1    4750 1850
+	0    1    1    0
+$EndComp
 $EndSCHEMATC

Commit message: ksch: fix error in codec supply
Parts:
- added C1, C10, C11, C12, C13, C16, C?: 10uF, symbol C_Small
- added C15, C19: 1uF, symbol C_Small
- added C17: 470pF, symbol C_Small
- added C18: 22uF, symbol C_Small
- added C2, C4, C5, C6, C7, C9: 0.1uF, symbol C_Small
- added J1: JMP, symbol JMP
- added R1: 33R, symbol R_Small
- added U2: WM8778-units, symbol WM8778-units
- added U4: AZ1117C, symbol AZ1117C
- added U5: TC1185, symbol TC1185
- renumbered C3 to C14, C1 to C3, C2 to C8, R1 to R2, R2 to R3, U2 to U3
Connections:
- net labels added: 3.3V, 5V, AGND
- net labels removed: 5.4V, 9V
- wire segments 17 -> 51
Other:
- note added: "3.3V LDO"
- note added: "5V LDO"
- note added: "9V Wall Supply"
- note added: "<200mOhm ESR"
- note added: "<3mm"
- note added: "CODEC Supply"
- note added: "Digital Ground to Analog Ground connenction"
- note added: "Reverse Polarity Protection?"
- note added: "Switching Regulator"
- note added: "additional filtering required?"
- note added: "caps against output or input ground?"
- note added: "only if supply is noisy"

Commit message: ksch: add uC power and programming pins
Parts:
- added C?: 0.1u, symbol C
- added C?: 4.7u, symbol C_Small
- added C? (x6): 100n, symbol C_Small
- added C?: 1u, symbol C
- added C?: 4.7u, symbol C
- added D?: D_Small_ALT, symbol D_Small_ALT
- added SW?: SW_Push, symbol SW_Push
- added U?: STM32F401RC, symbol STM32F401RC
Connections:
- net labels added: 3V_battery
- wire segments 51 -> 84
Other:
- note added: "unless implemented,\nconnect VBAT pin like this to 3.3v"

Commit message: ksch: add boot0 pin to switch
Connections:
- net labels added: BOOT
Changed lines of the file:
@@
 Text Label 6900 4100 1    60   ~ 0
 3.3V
-$Comp
-L GND #PWR?
-U 1 1 58D0B0AD
-P 7650 5550
-F 0 "#PWR?" H 7650 5300 50  0001 C CNN
-F 1 "GND" H 7650 5400 50  0000 C CNN
-F 2 "" H 7650 5550 50  0001 C CNN
-F 3 "" H 7650 5550 50  0001 C CNN
-	1    7650 5550
-	1    0    0    -1
-$EndComp
 Text Notes 6500 3850 0    60   ~ 0
 unless implemented,\nconnect VBAT pin like this to 3.3v
@@
 Connection ~ 2150 1550
 Connection ~ 2150 1750
+Text GLabel 7650 5550 0    60   Input ~ 0
+BOOT
 $EndSCHEMATC
