File: codec.sch (KiCad schematic (older format))
At the start: 3 parts, among them U1 WM8778

Commit message: ksch: add filter to both analog out channels
Parts:
- added C? (x2): 10uF, symbol CP
- added C? (x2): 4.7nF, symbol C_Small
- added R? (x4): 560, symbol R_Small
Connections:
- wire segments 0 -> 10
Other:
- note added: "implement better LPF + 2xmult, \nsee wolfson datasheet"
Changed lines of the file:
@@
 	1    0    0    -1
 $EndComp
+$Comp
+L R_Small R?
+U 1 1 590F46EC
+P 8400 5600
+F 0 "R?" V 8475 5550 50  0000 L CNN
+F 1 "560" V 8400 5525 50  0000 L CNN
+F 2 "" H 8400 5600 50  0001 C CNN
+F 3 "" H 8400 5600 50  0001 C CNN
+	1    8400 5600
+	0    1    1    0
+$EndComp
+$Comp
+L CP C?
+U 1 1 590F4BF4
+P 8050 5600
+F 0 "C?" H 8075 5700 50  0000 L CNN
+F 1 "10uF" H 8075 5500 50  0000 L CNN
+F 2 "" H 8088 5450 50  0001 C CNN
+F 3 "" H 8050 5600 50  0001 C CNN
+	1    8050 5600
+	0    -1   -1   0
+$EndComp
+$Comp
+L C_Small C?
+U 1 1 590F4CDD
+P 8550 5700
+F 0 "C?" H 8560 5770 50  0000 L CNN
+F 1 "4.7nF" H 8560 5620 50  0000 L CNN
+F 2 "" H 8550 5700 50  0001 C CNN
+F 3 "" H 8550 5700 50  0001 C CNN
+	1    8550 5700
+	1    0    0    -1
+$EndComp
+Wire Wire Line
+	7850 5600 7900 5600
+$Comp
+L AGND #PWR?
+U 1 1 590F584D
+P 8550 5850
+F 0 "#PWR?" H 8550 5600 50  0001 C CNN
+F 1 "AGND" H 8550 5700 50  0000 C CNN
+F 2 "" H 8550 5850 50  0000 C CNN
+F 3 "" H 8550 5850 50  0000 C CNN
+	1    8550 5850
+	1    0    0    -1
+$EndComp
+Wire Wire Line
+	8550 5850 8550 5800
+Wire Notes Line
+	7900 4525 7900 6125
+Wire Notes Line
+	7900 5325 8700 5325
+Wire Notes Line
+	8700 4525 8700 6125
+Wire Notes Line
+	8700 6125 7900 6125
+Text Notes 7900 4500 0    60   ~ 0
+implement better LPF + 2xmult, \nsee wolfson datasheet
+$Comp
+L R_Small R?
+U 1 1 59384C92
+P 8250 5700
+F 0 "R?" H 8250 5825 50  0000 L CNN
+F 1 "560" V 8300 5625 50  0000 L CNN
+F 2 "" H 8250 5700 50  0001 C CNN
+F 3 "" H 8250 5700 50  0001 C CNN
+	1    8250 5700
+	-1   0    0    1
+$EndComp
+$Comp
+L AGND #PWR?
+U 1 1 59384CD4
+P 8250 5850
+F 0 "#PWR?" H 8250 5600 50  0001 C CNN
+F 1 "AGND" H 8250 5700 50  0000 C CNN
+F 2 "" H 8250 5850 50  0000 C CNN
+F 3 "" H 8250 5850 50  0000 C CNN
+	1    8250 5850
+	1    0    0    -1
+$EndComp
+Wire Wire Line
+	8250 5850 8250 5800
+Wire Wire Line
+	8200 5600 8300 5600
+Connection ~ 8250 5600
+Wire Wire Line
+	8500 5600 8750 5600
+Connection ~ 8550 5600
+$Comp
+L R_Small R?
+U 1 1 59386657
+P 8400 4800
+F 0 "R?" V 8475 4750 50  0000 L CNN
+F 1 "560" V 8400 4725 50  0000 L CNN
+F 2 "" H 8400 4800 50  0001 C CNN
+F 3 "" H 8400 4800 50  0001 C CNN
+	1    8400 4800
+	0    1    1    0
+$EndComp
+$Comp
+L CP C?
+U 1 1 5938665D
+P 8050 4800
+F 0 "C?" H 8075 4900 50  0000 L CNN
+F 1 "10uF" H 8075 4700 50  0000 L CNN
+F 2 "" H 8088 4650 50  0001 C CNN
+F 3 "" H 8050 4800 50  0001 C CNN
+	1    8050 4800
+	0    -1   -1   0
+$EndComp
+$Comp
+L C_Small C?
+U 1 1 59386663
+P 8550 4900
+F 0 "C?" H 8560 4970 50  0000 L CNN
+F 1 "4.7nF" H 8560 4820 50  0000 L CNN
+F 2 "" H 8550 4900 50  0001 C CNN
+F 3 "" H 8550 4900 50  0001 C CNN
+	1    8550 4900
+	1    0    0    -1
+$EndComp
+$Comp
+L AGND #PWR?
+U 1 1 5938666A
+P 8550 5050
+F 0 "#PWR?" H 8550 4800 50  0001 C CNN
+F 1 "AGND" H 8550 4900 50  0000 C CNN
+F 2 "" H 8550 5050 50  0000 C CNN
+F 3 "" H 8550 5050 50  0000 C CNN
+	1    8550 5050
+	1    0    0    -1
+$EndComp
+Wire Wire Line
+	8550 5050 8550 5000
+Wire Notes Line
+	7900 4525 8700 4525
+$Comp
+L R_Small R?
+U 1 1 59386675
+P 8250 4900
+F 0 "R?" H 8250 5025 50  0000 L CNN
+F 1 "560" V 8300 4825 50  0000 L CNN
+F 2 "" H 8250 4900 50  0001 C CNN
+F 3 "" H 8250 4900 50  0001 C CNN
+	1    8250 4900
+	-1   0    0    1
+$EndComp
+$Comp
+L AGND #PWR?
+U 1 1 5938667B
+P 8250 5050
+F 0 "#PWR?" H 8250 4800 50  0001 C CNN
+F 1 "AGND" H 8250 4900 50  0000 C CNN
+F 2 "" H 8250 5050 50  0000 C CNN
+F 3 "" H 8250 5050 50  0000 C CNN
+	1    8250 5050
+	1    0    0    -1
+$EndComp
+Wire Wire Line
+	8250 5050 8250 5000
+Wire Wire Line
+	8200 4800 8300 4800
+Connection ~ 8250 4800
+Wire Wire Line
+	8500 4800 8750 4800
+Connection ~ 8550 4800
+Wire Wire Line
+	7850 4800 7900 4800
 $EndSCHEMATC
