File: controller.sch (KiCad schematic (older format))
At the start: 3 parts, among them U1 WM8778

Commit message: ksch: add uC power and programming pins
Parts:
- removed U1: WM8778, symbol WM8778
- removed U? (x2): WM8778-units, symbol WM8778-units
- added J?: CONN_01X04, symbol CONN_01X04
- added U?: STM32F401RC, symbol STM32F401RC
- added U?: WM8778-units, symbol WM8778-units
Connections:
- net labels added: GND
- net labels removed: 5V, AGND, DGND
- wire segments 0 -> 10
- no-connect marks 28 -> 0
Other:
- note removed: "HIGH: I2S Mode\nLOW: 2pin Mode\nFLOAT: Hardware Mode"
Changed lines of the file:
@@
 $Descr A4 11693 8268
 encoding utf-8
-Sheet 4 4
+Sheet 3 4
 Title ""
 Date ""
@@
 $EndDescr
 $Comp
-L WM8778 U1
-U 1 1 58B348AD
-P 4950 3250
-F 0 "U1" H 4700 4700 60  0000 C CNN
-F 1 "WM8778" H 4900 4200 60  0000 C CNN
-F 2 "" H 4700 3750 60  0000 C CNN
-F 3 "" H 4700 3750 60  0000 C CNN
-	1    4950 3250
-	1    0    0    -1
-$EndComp
-Text HLabel 4050 1950 0    60   Input ~ 0
-3.3V
-Text HLabel 4050 2150 0    60   Input ~ 0
-DGND
-Text HLabel 5850 1950 2    60   Input ~ 0
-5V
-Text HLabel 5850 2150 2    60   Input ~ 0
-AGND
-Text Notes 3750 2550 2    60   ~ 0
-HIGH: I2S Mode\nLOW: 2pin Mode\nFLOAT: Hardware Mode
-NoConn ~ 4050 2150
-NoConn ~ 4050 2600
-NoConn ~ 4050 2700
-NoConn ~ 4050 2800
-NoConn ~ 4050 3050
-NoConn ~ 4050 3150
-NoConn ~ 4050 3250
-NoConn ~ 4050 3350
-NoConn ~ 4050 3600
-NoConn ~ 4050 3700
-NoConn ~ 4050 3800
-NoConn ~ 4050 3900
-NoConn ~ 4050 4250
-NoConn ~ 4050 4550
-NoConn ~ 5850 4550
-NoConn ~ 5850 4450
-NoConn ~ 5850 4000
-NoConn ~ 5850 3900
-NoConn ~ 5850 3550
-NoConn ~ 5850 3400
-NoConn ~ 5850 3150
-NoConn ~ 5850 2950
-NoConn ~ 5850 2650
-NoConn ~ 5850 2450
-NoConn ~ 5850 2150
-NoConn ~ 5850 1950
-NoConn ~ 4050 2450
-NoConn ~ 4050 1950
-$Comp
-L WM8778-units U?
-U 2 1 58D0FD19
-P 7900 2800
-F 0 "U?" H 7600 3700 60  0000 C CNN
-F 1 "WM8778-units" H 7850 3250 60  0000 C CNN
-F 2 "" H 7650 2800 60  0000 C CNN
-F 3 "" H 7650 2800 60  0000 C CNN
-	2    7900 2800
+L STM32F401RC U?
+U 1 1 58D0F889
+P 3150 2800
+F 0 "U?" H 2800 3850 60  0000 C CNN
+F 1 "STM32F401RC" H 3150 1750 60  0000 C CNN
+F 2 "" H 3100 2750 60  0001 C CNN
+F 3 "" H 3100 2750 60  0001 C CNN
+	1    3150 2800
 	1    0    0    -1
 $EndComp
 $Comp
-L WM8778-units U?
-U 3 1 58D0FD94
-P 6950 5200
-F 0 "U?" H 6650 6100 60  0000 C CNN
-F 1 "WM8778-units" H 6900 5650 60  0000 C CNN
-F 2 "" H 6700 5200 60  0000 C CNN
-F 3 "" H 6700 5200 60  0000 C CNN
-	3    6950 5200
+L CONN_01X04 J?
+U 1 1 58D0F94B
+P 4900 2250
+F 0 "J?" H 4900 2500 50  0000 C CNN
+F 1 "CONN_01X04" V 5000 2250 50  0000 C CNN
+F 2 "" H 4900 2250 50  0001 C CNN
+F 3 "" H 4900 2250 50  0001 C CNN
+	1    4900 2250
 	1    0    0    -1
 $EndComp
+Wire Wire Line
+	4700 2100 4450 2100
+Wire Wire Line
+	4450 2100 4450 2050
+Text GLabel 1200 1100 0    60   Input ~ 0
+3.3V
+Wire Wire Line
+	1200 1100 1350 1100
+Text Label 1350 1100 0    60   ~ 0
+3.3V
+Text Label 4450 2050 0    60   ~ 0
+3.3V
+Wire Wire Line
+	4700 2200 4100 2200
+Wire Wire Line
+	4100 2200 4100 2150
+Wire Wire Line
+	4100 2150 3900 2150
+Wire Wire Line
+	4700 2300 4450 2300
+Wire Wire Line
+	4450 2300 4450 2450
+$Comp
+L GND #PWR?
+U 1 1 58D0FA65
+P 4450 2450
+F 0 "#PWR?" H 4450 2200 50  0001 C CNN
+F 1 "GND" H 4450 2300 50  0000 C CNN
+F 2 "" H 4450 2450 50  0001 C CNN
+F 3 "" H 4450 2450 50  0001 C CNN
+	1    4450 2450
+	1    0    0    -1
+$EndComp
+Wire Wire Line
+	4700 2400 3900 2400
+$Comp
+L WM8778-units U?
+U 2 1 58D101B0
+P 8800 3250
+F 0 "U?" H 8500 4150 60  0000 C CNN
+F 1 "WM8778-units" H 8750 3700 60  0000 C CNN
+F 2 "" H 8550 3250 60  0000 C CNN
+F 3 "" H 8550 3250 60  0000 C CNN
+	2    8800 3250
+	1    0    0    -1
+$EndComp
+Wire Wire Line
+	7750 2450 7900 2450
+Text Label 7750 2450 0    60   ~ 0
+3.3V
 $EndSCHEMATC

Commit message: ksch: add I2S interface connections
Parts:
- added SW?: SW_SPDT, symbol SW_SPDT
- added U? (x2): STM32F401RC, symbol STM32F401RC
Connections:
- net labels added: I2S2_CK, I2S2_SD, I2S2_WS, I2S3_CK, I2S3_SD, I2S3_WS, MCLK, SDIO_CMD
- wire segments 10 -> 17
Other:
- note added: "stopping will power down adc/dac, restarting powers them up again\nvolume needs to be updated for correct settings again!"
- note added: "temporary HIGH -> I2S mode"
- note added: "temporary LOW -> 16bit"
- note added: "temporary LOW -> no de-emphasis"
- note added: "temporary left midrail.\n-> hardware control"
Changed lines of the file:
@@
 LIBS:zetex
 LIBS:Zilog
+LIBS:looper-cache
 EELAYER 25 0
 EELAYER END
@@
 L STM32F401RC U?
 U 1 1 58D0F889
-P 3150 2800
-F 0 "U?" H 2800 3850 60  0000 C CNN
-F 1 "STM32F401RC" H 3150 1750 60  0000 C CNN
-F 2 "" H 3100 2750 60  0001 C CNN
-F 3 "" H 3100 2750 60  0001 C CNN
-	1    3150 2800
+P 2550 1600
+F 0 "U?" H 2200 2650 60  0000 C CNN
+F 1 "STM32F401RC" H 2550 550 60  0000 C CNN
+F 2 "" H 2500 1550 60  0001 C CNN
+F 3 "" H 2500 1550 60  0001 C CNN
+	1    2550 1600
 	1    0    0    -1
 $EndComp
@@
 L CONN_01X04 J?
 U 1 1 58D0F94B
-P 4900 2250
-F 0 "J?" H 4900 2500 50  0000 C CNN
-F 1 "CONN_01X04" V 5000 2250 50  0000 C CNN
-F 2 "" H 4900 2250 50  0001 C CNN
-F 3 "" H 4900 2250 50  0001 C CNN
-	1    4900 2250
+P 4300 1050
+F 0 "J?" H 4300 1300 50  0000 C CNN
+F 1 "CONN_01X04" V 4400 1050 50  0000 C CNN
+F 2 "" H 4300 1050 50  0001 C CNN
+F 3 "" H 4300 1050 50  0001 C CNN
+	1    4300 1050
 	1    0    0    -1
 $EndComp
 Wire Wire Line
-	4700 2100 4450 2100
+	4100 900  3850 900
 Wire Wire Line
-	4450 2100 4450 2050
-Text GLabel 1200 1100 0    60   Input ~ 0
+	3850 900  3850 850
+Text GLabel 1100 950  0    60   Input ~ 0
 3.3V
 Wire Wire Line
-	1200 1100 1350 1100
-Text Label 1350 1100 0    60   ~ 0
+	1100 950  1250 950
+Text Label 1250 950  0    60   ~ 0
 3.3V
-Text Label 4450 2050 0    60   ~ 0
+Text Label 3850 850  0    60   ~ 0
 3.3V
 Wire Wire Line
-	4700 2200 4100 2200
+	4100 1000 3500 1000
 Wire Wire Line
-	4100 2200 4100 2150
+	3500 1000 3500 950
 Wire Wire Line
-	4100 2150 3900 2150
+	3500 950  3300 950
 Wire Wire Line
-	4700 2300 4450 2300
+	4100 1100 3850 1100
 Wire Wire Line
-	4450 2300 4450 2450
+	3850 1100 3850 1250
 $Comp
 L GND #PWR?
 U 1 1 58D0FA65
-P 4450 2450
-F 0 "#PWR?" H 4450 2200 50  0001 C CNN
-F 1 "GND" H 4450 2300 50  0000 C CNN
-F 2 "" H 4450 2450 50  0001 C CNN
-F 3 "" H 4450 2450 50  0001 C CNN
-	1    4450 2450
+P 3850 1250
+F 0 "#PWR?" H 3850 1000 50  0001 C CNN
+F 1 "GND" H 3850 1100 50  0000 C CNN
+F 2 "" H 3850 1250 50  0001 C CNN
+F 3 "" H 3850 1250 50  0001 C CNN
+	1    3850 1250
 	1    0    0    -1
 $EndComp
 Wire Wire Line
-	4700 2400 3900 2400
+	4100 1200 3300 1200
 $Comp
 L WM8778-units U?
 U 2 1 58D101B0
-P 8800 3250
-F 0 "U?" H 8500 4150 60  0000 C CNN
-F 1 "WM8778-units" H 8750 3700 60  0000 C CNN
-F 2 "" H 8550 3250 60  0000 C CNN
-F 3 "" H 8550 3250 60  0000 C CNN
-	2    8800 3250
+P 8700 2350
+F 0 "U?" H 8400 3250 60  0000 C CNN
+F 1 "WM8778-units" H 8650 2800 60  0000 C CNN
+F 2 "" H 8450 2350 60  0000 C CNN
+F 3 "" H 8450 2350 60  0000 C CNN
+	2    8700 2350
 	1    0    0    -1
 $EndComp
 Wire Wire Line
-	7750 2450 7900 2450
-Text Label 7750 2450 0    60   ~ 0
+	7650 1550 7800 1550
+Text Label 7650 1550 0    60   ~ 0
 3.3V
+$Comp
+L STM32F401RC U?
+U 3 1 58FD347E
+P 2550 5800
+F 0 "U?" H 2200 6850 60  0000 C CNN
+F 1 "STM32F401RC" H 2550 4750 60  0000 C CNN
+F 2 "" H 2500 5750 60  0001 C CNN
+F 3 "" H 2500 5750 60  0001 C CNN
+	3    2550 5800
+	1    0    0    -1
+$EndComp
+Wire Wire Line
+	6200 6450 3300 6450
+Wire Wire Line
+	6200 2150 6200 2700
+Wire Wire Line
+	6200 2700 6200 6450
+Wire Wire Line
+	6200 2150 7800 2150
+Wire Wire Line
+	7800 2700 6200 2700
+Connection ~ 6200 2700
+Text Notes 3650 6550 0    60   ~ 0
+stopping will power down adc/dac, restarting powers them up again\nvolume needs to be updated for correct settings again!
+Text Label 3350 6450 0    60   ~ 0
+MCLK
+Wire Wire Line
+	1800 1750 1600 1750
+Text Label 1600 1750 2    60   ~ 0
+I2S3_WS
+$Comp
+L STM32F401RC U?
+U 2 1 58FD4D8F
+P 2550 3700
+F 0 "U?" H 2200 4750 60  0000 C CNN
+F 1 "STM32F401RC" H 2550 2650 60  0000 C CNN
+F 2 "" H 2500 3650 60  0001 C CNN
+F 3 "" H 2500 3650 60  0001 C CNN
+	2    2550 3700
+	1    0    0    -1
+$EndComp
+Text Label 3300 2800 0    60   ~ 0
+SDIO_CMD
+Wire Wire Line
+	1800 3300 1450 3300
+$Comp
+L SW_SPDT SW?
+U 1 1 58FD6197
+P 1250 3300
+F 0 "SW?" H 1250 3470 50  0000 C CNN
+F 1 "SW_SPDT" H 1250 3100 50  0000 C CNN
+F 2 "" H 1250 3300 50  0001 C CNN
+F 3 "" H 1250 3300 50  0001 C CNN
+	1    1250 3300
+	-1   0    0    1
+$EndComp
+Text Label 1050 3200 2    60   ~ 0
+3.3V
+Text Label 1050 3400 2    60   ~ 0
+GND
+Text Label 1800 3550 2    60   ~ 0
+I2S3_CK
+Text Label 1800 4100 2    60   ~ 0
+I2S3_SD
+Text Label 3300 3850 0    60   ~ 0
+I2S2_WS
+Text Label 3300 3550 0    60   ~ 0
+I2S2_CK
+Text Label 3300 3050 0    60   ~ 0
+I2S2_SD
+Text Label 7800 2250 2    60   ~ 0
+I2S3_CK
+Text Label 7800 2350 2    60   ~ 0
+I2S3_WS
+Text Label 7800 2450 2    60   ~ 0
+I2S3_SD
+Text Label 7800 2800 2    60   ~ 0
+I2S2_CK
+Text Label 7800 2900 2    60   ~ 0
+I2S2_WS
+Text Label 7800 3000 2    60   ~ 0
+I2S2_SD
+Text Notes 7750 1600 2    60   ~ 0
+temporary left midrail.\n-> hardware control
+Text Notes 7800 1700 2    60   ~ 0
+temporary HIGH -> I2S mode
+Text Notes 7800 1800 2    60   ~ 0
+temporary LOW -> 16bit
+Text Notes 7800 1900 2    60   ~ 0
+temporary LOW -> no de-emphasis
 $EndSCHEMATC

Commit message: ksch: use i2s2 and i2s3 for codec
Parts:
- SW?: value SW_SPDT -> RAM~FLASH
Connections:
- net labels added: I2S2_MCK, I2S3_MCK, to_*MCLK
- wire segments 17 -> 18
Other:
- note added: "decide on this or stm being i2s master"
Changed lines of the file:
@@
 encoding utf-8
 Sheet 3 4
-Title ""
+Title "FG_27"
 Date ""
-Rev ""
-Comp ""
+Rev "3.87"
+Comp "Jonathan Halmen"
 Comment1 ""
 Comment2 ""
@@
 	6200 6450 3300 6450
 Wire Wire Line
-	6200 2150 6200 2700
-Wire Wire Line
-	6200 2700 6200 6450
-Wire Wire Line
 	6200 2150 7800 2150
 Wire Wire Line
 	7800 2700 6200 2700
-Connection ~ 6200 2700
 Text Notes 3650 6550 0    60   ~ 0
 stopping will power down adc/dac, restarting powers them up again\nvolume needs to be updated for correct settings again!
@@
 P 1250 3300
 F 0 "SW?" H 1250 3470 50  0000 C CNN
-F 1 "SW_SPDT" H 1250 3100 50  0000 C CNN
+F 1 "RAM~FLASH" H 1250 3100 50  0000 C CNN
 F 2 "" H 1250 3300 50  0001 C CNN
 F 3 "" H 1250 3300 50  0001 C CNN
@@
 Text Notes 7800 1900 2    60   ~ 0
 temporary LOW -> no de-emphasis
+Wire Notes Line
+	3300 6250 7100 6250
+Wire Notes Line
+	7100 6250 7100 6650
+Wire Notes Line
+	7100 6650 3300 6650
+Wire Notes Line
+	3300 6650 3300 6250
+Text Label 6200 6100 0    60   ~ 0
+to_*MCLK
+Text Notes 4350 6200 0    60   ~ 0
+decide on this or stm being i2s master
+Wire Wire Line
+	6200 6450 6200 6100
+Wire Wire Line
+	1800 6450 1550 6450
+Text Label 1550 6450 2    60   ~ 0
+I2S2_MCK
+Wire Wire Line
+	1800 6700 1550 6700
+Text Label 1550 6700 2    60   ~ 0
+I2S3_MCK
+Text Label 6200 2150 0    60   ~ 0
+I2S3_MCK
+Text Label 6200 2700 0    60   ~ 0
+I2S2_MCK
 $EndSCHEMATC

Commit message: ksch: change to use i2s2 bidirectional, free i2s3
Connections:
- net labels added: I2S2ext
- net labels removed: I2S3_CK, I2S3_MCK, I2S3_SD, I2S3_WS, MCLK, to_*MCLK
- wire segments 18 -> 20
Other:
- note removed: "decide on this or stm being i2s master"
- note removed: "stopping will power down adc/dac, restarting powers them up again\nvolume needs to be updated for correct settings again!"
Changed lines of the file:
@@
 $EndComp
 Wire Wire Line
-	6200 6450 3300 6450
-Wire Wire Line
-	6200 2150 7800 2150
-Wire Wire Line
-	7800 2700 6200 2700
-Text Notes 3650 6550 0    60   ~ 0
-stopping will power down adc/dac, restarting powers them up again\nvolume needs to be updated for correct settings again!
-Text Label 3350 6450 0    60   ~ 0
-MCLK
-Wire Wire Line
-	1800 1750 1600 1750
-Text Label 1600 1750 2    60   ~ 0
-I2S3_WS
+	6200 2700 7800 2700
 $Comp
 L STM32F401RC U?
@@
 Text Label 1050 3400 2    60   ~ 0
 GND
-Text Label 1800 3550 2    60   ~ 0
-I2S3_CK
-Text Label 1800 4100 2    60   ~ 0
-I2S3_SD
 Text Label 3300 3850 0    60   ~ 0
 I2S2_WS
@@
 Text Label 3300 3050 0    60   ~ 0
 I2S2_SD
-Text Label 7800 2250 2    60   ~ 0
-I2S3_CK
-Text Label 7800 2350 2    60   ~ 0
-I2S3_WS
 Text Label 7800 2450 2    60   ~ 0
-I2S3_SD
-Text Label 7800 2800 2    60   ~ 0
+I2S2ext
+Text Label 6200 2800 0    60   ~ 0
 I2S2_CK
-Text Label 7800 2900 2    60   ~ 0
+Text Label 6200 2900 0    60   ~ 0
 I2S2_WS
 Text Label 7800 3000 2    60   ~ 0
@@
 Text Notes 7800 1900 2    60   ~ 0
 temporary LOW -> no de-emphasis
-Wire Notes Line
-	3300 6250 7100 6250
-Wire Notes Line
-	7100 6250 7100 6650
-Wire Notes Line
-	7100 6650 3300 6650
-Wire Notes Line
-	3300 6650 3300 6250
-Text Label 6200 6100 0    60   ~ 0
-to_*MCLK
-Text Notes 4350 6200 0    60   ~ 0
-decide on this or stm being i2s master
-Wire Wire Line
-	6200 6450 6200 6100
-Wire Wire Line
-	1800 6450 1550 6450
-Text Label 1550 6450 2    60   ~ 0
+Text Label 1800 6450 2    60   ~ 0
+I2S2_MCK
+Text Label 6200 2700 0    60   ~ 0
 I2S2_MCK
 Wire Wire Line
-	1800 6700 1550 6700
-Text Label 1550 6700 2    60   ~ 0
-I2S3_MCK
-Text Label 6200 2150 0    60   ~ 0
-I2S3_MCK
-Text Label 6200 2700 0    60   ~ 0
-I2S2_MCK
+	7200 2700 7200 2150
+Connection ~ 7200 2700
+Wire Wire Line
+	7200 2150 7800 2150
+Wire Wire Line
+	7800 2800 6200 2800
+Wire Wire Line
+	6200 2900 7800 2900
+Wire Wire Line
+	7250 2800 7250 2250
+Wire Wire Line
+	7250 2250 7800 2250
+Connection ~ 7250 2800
+Wire Wire Line
+	7300 2900 7300 2350
+Wire Wire Line
+	7300 2350 7800 2350
+Connection ~ 7300 2900
+Text Label 1800 5400 2    60   ~ 0
+I2S2ext
 $EndSCHEMATC

Commit message: ksch: add codec control interface as i2c1
Connections:
- net labels added: BOOT, I2C1_SCL, I2C1_SDA
- wire segments 20 -> 24
Other:
- note removed: "temporary HIGH -> I2S mode"
- note removed: "temporary LOW -> 16bit"
- note removed: "temporary LOW -> no de-emphasis"
- note removed: "temporary left midrail.\n-> hardware control"
Changed lines of the file:
@@
 Wire Wire Line
 	7650 1550 7800 1550
-Text Label 7650 1550 0    60   ~ 0
-3.3V
 $Comp
 L STM32F401RC U?
@@
 Text Label 3300 3050 0    60   ~ 0
 I2S2_SD
-Text Label 7800 2450 2    60   ~ 0
+Text Label 7800 3000 2    60   ~ 0
 I2S2ext
 Text Label 6200 2800 0    60   ~ 0
@@
 Text Label 6200 2900 0    60   ~ 0
 I2S2_WS
-Text Label 7800 3000 2    60   ~ 0
+Text Label 7800 2450 2    60   ~ 0
 I2S2_SD
-Text Notes 7750 1600 2    60   ~ 0
-temporary left midrail.\n-> hardware control
-Text Notes 7800 1700 2    60   ~ 0
-temporary HIGH -> I2S mode
-Text Notes 7800 1800 2    60   ~ 0
-temporary LOW -> 16bit
-Text Notes 7800 1900 2    60   ~ 0
-temporary LOW -> no de-emphasis
 Text Label 1800 6450 2    60   ~ 0
 I2S2_MCK
@@
 	7200 2150 7800 2150
 Wire Wire Line
-	7800 2800 6200 2800
+	6200 2800 7800 2800
 Wire Wire Line
 	6200 2900 7800 2900
@@
 Text Label 1800 5400 2    60   ~ 0
 I2S2ext
+$Comp
+L GND #PWR?
+U 1 1 593872BF
+P 7650 1550
+F 0 "#PWR?" H 7650 1300 50  0001 C CNN
+F 1 "GND" H 7650 1400 50  0000 C CNN
+F 2 "" H 7650 1550 50  0001 C CNN
+F 3 "" H 7650 1550 50  0001 C CNN
+	1    7650 1550
+	1    0    0    -1
+$EndComp
+Wire Wire Line
+	7800 1700 7750 1700
+Wire Wire Line
+	7750 1700 7750 1550
+Connection ~ 7750 1550
+Wire Wire Line
+	7800 1800 7400 1800
+Wire Wire Line
+	7800 1900 7400 1900
+Text Label 7400 1800 2    60   ~ 0
+I2C1_SDA
+Text Label 7400 1900 2    60   ~ 0
+I2C1_SCL
+Text Label 1800 4600 2    60   ~ 0
+I2C1_SDA
+Text Label 1800 4350 2    60   ~ 0
+I2C1_SCL
+Text GLabel 1600 3300 1    60   Input ~ 0
+BOOT
 $EndSCHEMATC

Commit message: ksch: add stuff that isn't on soldered prototype yet
this hopefully completes the rev. A schematics
Parts:
- added C1: 0.1u, Capacitors_SMD:C_0805_HandSoldering, symbol C_Small
- added C10: 4.7u, Capacitors_SMD:C_0805_HandSoldering, symbol C_Small
- added C11: 10u, Capacitors_SMD:C_0805_HandSoldering, symbol C_Small
- added J302: Micro_SD_Card_Det, footprints:SD-503182_Molex_micro_SD_HandSolder, symbol Micro_SD_Card_Det
- added J4: UART, Pin_Headers:Pin_Header_Straight_1x02_Pitch2.54mm, symbol CONN_01X02
- added R1, R2, R3, R4: 4.7k, Resistors_THT:R_Axial_DIN0207_L6.3mm_D2.5mm_P7.62mm_Horizontal, symbol R_Small
- added RV1: pot_in_l, Potentiometers:Potentiometer_WirePads_Small, symbol POT
- added RV2: pot_in_r, Potentiometers:Potentiometer_WirePads_Small, symbol POT
- added RV3: pot_out, Potentiometers:Potentiometer_WirePads_Small, symbol POT
- added SW1: start, Buttons_Switches_THT:SW_PUSH_6mm, symbol SW_Push
- added SW2: stop, Buttons_Switches_THT:SW_PUSH_6mm, symbol SW_Push
- added SW3: Rotary_Encoder_Switch, footprints:EN11-HSM, symbol Rotary_Encoder_Switch
- added U1: lcd, Socket_Strips:Socket_Strip_Straight_1x04_Pitch2.54mm, symbol lcd
- added Y1: CSTLS4M00G53-B0, Crystals:Resonator_muRata_CSTLSxxxG-3pin_w8.0mm_h3.0mm, symbol Resonator_Small
- J301: renamed from J?; value CONN_01X04 -> programming header; footprint (none) -> Pin_Headers:Pin_Header_Straight_1x04_Pitch2.54mm
- SW301: renamed from SW?; footprint (none) -> Buttons_Switches_THT:SW_Micro_SPST
- U201: renamed from U?; footprint (none) -> footprints:SSOP-28_5.3x10.2mm_Pitch0.65mm_HandSolder
- U205: renamed from U?; footprint (none) -> footprints:LQFP-64_10x10mm_Pitch0.5mm_HandSolder
Connections:
- net labels added: ADC1_IN5, ADC1_IN6, ADC1_IN7, DISP_SCL, DISP_SDA, SDIO_CK, SDIO_D0, SDIO_D1, SDIO_D2, SDIO_D3, SDdetect, TIM2_CH1, TIM2_CH2, USART1_RX, USART1_TX, rot_but, stomp_start, stomp_stop
- wire segments 24 -> 60
Other:
- note added: "CE low -> I2C address: 0x34"
- note added: "DISP is on I2C2 periph"
- note added: "MODE low -> I2C mode"
- note added: "Volume Control"
- note added: "looper control"
