File: controller.sch (KiCad schematic (older format))
At the start: 21 parts, among them J301 programming header, J302 Micro_SD_Card_Det, J4 UART, SW1 start, SW2 stop, SW3 Rotary_Encoder_Switch, SW301 RAM~FLASH, U1 lcd, U201 WM8778-units, U205 STM32F401RC, Y1 CSTLS4M00G53-B0

Commit message: ksch: reannotate schematics to have a single style of part-naming
Parts:
- renumbered C10 to C31, C11 to C32, C1 to C33, J4 to J2, J301 to J3, J302 to J4, R1 to R4, R2 to R5, R3 to R6, R4 to R7, SW301 to SW2, SW1 to SW3, SW2 to SW4, SW3 to SW5, U201 to U1, U205 to U5, U1 to U6
Changed lines of the file:
@@
 $EndDescr
 $Comp
-L STM32F401RC U205
+L STM32F401RC U5
 U 1 1 58D0F889
 P 2550 1600
-F 0 "U205" H 2200 2650 60  0000 C CNN
+F 0 "U5" H 2200 2650 60  0000 C CNN
 F 1 "STM32F401RC" H 2550 550 60  0000 C CNN
 F 2 "footprints:LQFP-64_10x10mm_Pitch0.5mm_HandSolder" H 2500 1550 60  0001 C CNN
@@
 $EndComp
 $Comp
-L CONN_01X04 J301
+L CONN_01X04 J3
 U 1 1 58D0F94B
 P 4300 1050
-F 0 "J301" H 4300 1300 50  0000 C CNN
+F 0 "J3" H 4300 1300 50  0000 C CNN
 F 1 "programming header" V 4400 1050 50  0000 C CNN
 F 2 "Pin_Headers:Pin_Header_Straight_1x04_Pitch2.54mm" H 4300 1050 50  0001 C CNN
@@
 	3850 1100 3850 1250
 $Comp
-L GND #PWR0301
+L GND #PWR023
 U 1 1 58D0FA65
 P 3850 1250
-F 0 "#PWR0301" H 3850 1000 50  0001 C CNN
+F 0 "#PWR023" H 3850 1000 50  0001 C CNN
 F 1 "GND" H 3850 1100 50  0000 C CNN
 F 2 "" H 3850 1250 50  0001 C CNN
@@
 	4100 1200 3300 1200
 $Comp
-L WM8778-units U201
+L WM8778-units U1
 U 2 1 58D101B0
 P 8700 2350
-F 0 "U201" H 8400 3250 60  0000 C CNN
+F 0 "U1" H 8400 3250 60  0000 C CNN
 F 1 "WM8778-units" H 8650 2800 60  0000 C CNN
 F 2 "footprints:SSOP-28_5.3x10.2mm_Pitch0.65mm_HandSolder" H 8450 2350 60  0001 C CNN
@@
 	7650 1550 7800 1550
 $Comp
-L STM32F401RC U205
+L STM32F401RC U5
 U 3 1 58FD347E
 P 2550 5800
-F 0 "U205" H 2200 6850 60  0000 C CNN
+F 0 "U5" H 2200 6850 60  0000 C CNN
 F 1 "STM32F401RC" H 2550 4750 60  0000 C CNN
 F 2 "footprints:LQFP-64_10x10mm_Pitch0.5mm_HandSolder" H 2500 5750 60  0001 C CNN
@@
 	6700 2700 7800 2700
 $Comp
-L STM32F401RC U205
+L STM32F401RC U5
 U 2 1 58FD4D8F
 P 2550 3700
-F 0 "U205" H 2200 4750 60  0000 C CNN
+F 0 "U5" H 2200 4750 60  0000 C CNN
 F 1 "STM32F401RC" H 2550 2650 60  0000 C CNN
 F 2 "footprints:LQFP-64_10x10mm_Pitch0.5mm_HandSolder" H 2500 3650 60  0001 C CNN
@@
 	1800 3300 1450 3300
 $Comp
-L SW_SPDT SW301
+L SW_SPDT SW2
 U 1 1 58FD6197
 P 1250 3300
-F 0 "SW301" H 1250 3470 50  0000 C CNN
+F 0 "SW2" H 1250 3470 50  0000 C CNN
 F 1 "RAM~FLASH" H 1250 3100 50  0000 C CNN
 F 2 "Buttons_Switches_THT:SW_Micro_SPST" H 1250 3300 50  0001 C CNN
@@
 I2S2ext
 $Comp
-L GND #PWR0302
+L GND #PWR027
 U 1 1 593872BF
 P 7650 1550
-F 0 "#PWR0302" H 7650 1300 50  0001 C CNN
+F 0 "#PWR027" H 7650 1300 50  0001 C CNN
 F 1 "GND" H 7650 1400 50  0000 C CNN
 F 2 "" H 7650 1550 50  0001 C CNN
@@
 CE low -> I2C address: 0x34
 $Comp
-L Micro_SD_Card_Det J302
+L Micro_SD_Card_Det J4
 U 1 1 59C768AC
 P 8300 4250
-F 0 "J302" H 8250 5067 50  0000 C CNN
+F 0 "J4" H 8250 5067 50  0000 C CNN
 F 1 "Micro_SD_Card_Det" H 8250 4976 50  0000 C CNN
 F 2 "footprints:SD-503182_Molex_micro_SD_HandSolder" H 10350 4950 50  0001 C CNN
@@
 $EndComp
 $Comp
-L R_Small R3
+L R_Small R6
 U 1 1 59C79ED4
 P 7150 1650
-F 0 "R3" H 7209 1696 50  0000 L CNN
+F 0 "R6" H 7209 1696 50  0000 L CNN
 F 1 "4.7k" H 7209 1605 50  0000 L CNN
 F 2 "Resistors_THT:R_Axial_DIN0207_L6.3mm_D2.5mm_P7.62mm_Horizontal" H 7150 1650 50  0001 C CNN
@@
 $EndComp
 $Comp
-L R_Small R2
+L R_Small R5
 U 1 1 59C79F42
 P 6850 1650
-F 0 "R2" H 6909 1696 50  0000 L CNN
+F 0 "R5" H 6909 1696 50  0000 L CNN
 F 1 "4.7k" H 6909 1605 50  0000 L CNN
 F 2 "Resistors_THT:R_Axial_DIN0207_L6.3mm_D2.5mm_P7.62mm_Horizontal" H 6850 1650 50  0001 C CNN
@@
 	9100 4750 9150 4750
 $Comp
-L GND #PWR01
+L GND #PWR031
 U 1 1 59C7A31E
 P 9150 4750
-F 0 "#PWR01" H 9150 4500 50  0001 C CNN
+F 0 "#PWR031" H 9150 4500 50  0001 C CNN
 F 1 "GND" H 9150 4600 50  0000 C CNN
 F 2 "" H 9150 4750 50  0001 C CNN
@@
 	7400 4750 7350 4750
 $Comp
-L GND #PWR02
+L GND #PWR026
 U 1 1 59C7AD06
 P 7350 4750
-F 0 "#PWR02" H 7350 4500 50  0001 C CNN
+F 0 "#PWR026" H 7350 4500 50  0001 C CNN
 F 1 "GND" H 7350 4600 50  0000 C CNN
 F 2 "" H 7350 4750 50  0001 C CNN
@@
 	6700 4650 7400 4650
 $Comp
-L R_Small R1
+L R_Small R4
 U 1 1 59C7AE61
 P 6800 4550
-F 0 "R1" H 6859 4596 50  0000 L CNN
+F 0 "R4" H 6859 4596 50  0000 L CNN
 F 1 "4.7k" H 6859 4505 50  0000 L CNN
 F 2 "Resistors_THT:R_Axial_DIN0207_L6.3mm_D2.5mm_P7.62mm_Horizontal" H 6800 4550 50  0001 C CNN
@@
 GND
 $Comp
-L Rotary_Encoder_Switch SW3
+L Rotary_Encoder_Switch SW5
 U 1 1 59C7C119
 P 8350 5600
-F 0 "SW3" H 8350 5967 50  0000 C CNN
+F 0 "SW5" H 8350 5967 50  0000 C CNN
 F 1 "Rotary_Encoder_Switch" H 8350 5876 50  0000 C CNN
 F 2 "footprints:EN11-HSM" H 8250 5760 50  0001 C CNN
@@
 $EndComp
 $Comp
-L GND #PWR03
+L GND #PWR028
 U 1 1 59C7C7A0
 P 7950 5600
-F 0 "#PWR03" H 7950 5350 50  0001 C CNN
+F 0 "#PWR028" H 7950 5350 50  0001 C CNN
 F 1 "GND" H 7950 5450 50  0000 C CNN
 F 2 "" H 7950 5600 50  0001 C CNN
@@
 	8050 5600 7950 5600
 $Comp
-L GND #PWR04
+L GND #PWR030
 U 1 1 59C7C878
 P 8700 5700
-F 0 "#PWR04" H 8700 5450 50  0001 C CNN
+F 0 "#PWR030" H 8700 5450 50  0001 C CNN
 F 1 "GND" H 8700 5550 50  0000 C CNN
 F 2 "" H 8700 5700 50  0001 C CNN
@@
 TIM2_CH2
 $Comp
-L R_Small R4
+L R_Small R7
 U 1 1 59C7D0FB
 P 8900 5400
-F 0 "R4" H 8959 5446 50  0000 L CNN
+F 0 "R7" H 8959 5446 50  0000 L CNN
 F 1 "4.7k" H 8959 5355 50  0000 L CNN
 F 2 "Resistors_THT:R_Axial_DIN0207_L6.3mm_D2.5mm_P7.62mm_Horizontal" H 8900 5400 50  0001 C CNN
@@
 3.3V
 $Comp
-L C_Small C1
+L C_Small C33
 U 1 1 59C7D973
 P 8900 5600
-F 0 "C1" H 8992 5646 50  0000 L CNN
+F 0 "C33" H 8992 5646 50  0000 L CNN
 F 1 "0.1u" H 8992 5555 50  0000 L CNN
 F 2 "Capacitors_SMD:C_0805_HandSoldering" H 8900 5600 50  0001 C CNN
@@
 Connection ~ 8900 5500
 $Comp
-L lcd U1
+L lcd U6
 U 1 1 59C7E596
 P 8700 6350
-F 0 "U1" H 8900 6000 60  0000 R CNN
+F 0 "U6" H 8900 6000 60  0000 R CNN
 F 1 "lcd" H 8850 6600 60  0000 R CNN
 F 2 "Socket_Strips:Socket_Strip_Straight_1x04_Pitch2.54mm" H 8400 6400 60  0001 C CNN
@@
 	8000 6200 8200 6200
 $Comp
-L GND #PWR05
+L GND #PWR029
 U 1 1 59C7EAD2
 P 8100 6200
-F 0 "#PWR05" H 8100 5950 50  0001 C CNN
+F 0 "#PWR029" H 8100 5950 50  0001 C CNN
 F 1 "GND" H 8100 6050 50  0000 C CNN
 F 2 "" H 8100 6200 50  0001 C CNN
@@
 	5150 3000 5250 3000
 $Comp
-L GND #PWR06
+L GND #PWR024
 U 1 1 59C7F568
 P 5200 3000
-F 0 "#PWR06" H 5200 2750 50  0001 C CNN
+F 0 "#PWR024" H 5200 2750 50  0001 C CNN
 F 1 "GND" H 5200 2850 50  0000 C CNN
 F 2 "" H 5200 3000 50  0001 C CNN
@@
 Volume Control
 $Comp
-L SW_Push SW1
+L SW_Push SW3
 U 1 1 59C8045B
 P 5050 3950
-F 0 "SW1" H 5050 4235 50  0000 C CNN
+F 0 "SW3" H 5050 4235 50  0000 C CNN
 F 1 "start" H 5050 4144 50  0000 C CNN
 F 2 "Buttons_Switches_THT:SW_PUSH_6mm" H 5050 4150 50  0001 C CNN
@@
 $EndComp
 $Comp
-L SW_Push SW2
+L SW_Push SW4
 U 1 1 59C804E7
 P 5050 4300
-F 0 "SW2" H 5050 4585 50  0000 C CNN
+F 0 "SW4" H 5050 4585 50  0000 C CNN
 F 1 "stop" H 5050 4494 50  0000 C CNN
 F 2 "Buttons_Switches_THT:SW_PUSH_6mm" H 5050 4500 50  0001 C CNN
@@
 Connection ~ 5250 4300
 $Comp
-L GND #PWR07
+L GND #PWR025
 U 1 1 59C805DE
 P 5250 4400
-F 0 "#PWR07" H 5250 4150 50  0001 C CNN
+F 0 "#PWR025" H 5250 4150 50  0001 C CNN
 F 1 "GND" H 5250 4250 50  0000 C CNN
 F 2 "" H 5250 4400 50  0001 C CNN
@@
 USART1_RX
 $Comp
-L CONN_01X02 J4
+L CONN_01X02 J2
 U 1 1 59C92584
 P 3950 2100
-F 0 "J4" H 4028 2141 50  0000 L CNN
+F 0 "J2" H 4028 2141 50  0000 L CNN
 F 1 "UART" H 4028 2050 50  0000 L CNN
 F 2 "Pin_Headers:Pin_Header_Straight_1x02_Pitch2.54mm" H 3950 2100 50  0001 C CNN
@@
 	3300 2150 3750 2150
 $Comp
-L C_Small C11
+L C_Small C32
 U 1 1 59C92F89
 P 7950 6150
-F 0 "C11" H 8100 6100 50  0000 R CNN
+F 0 "C32" H 8100 6100 50  0000 R CNN
 F 1 "10u" H 8150 6200 50  0000 R CNN
 F 2 "Capacitors_SMD:C_0805_HandSoldering" H 7950 6150 50  0001 C CNN
@@
 Connection ~ 8100 6200
 $Comp
-L C_Small C10
+L C_Small C31
 U 1 1 59C93510
 P 6950 4250
-F 0 "C10" H 7100 4200 50  0000 R CNN
+F 0 "C31" H 7100 4200 50  0000 R CNN
 F 1 "4.7u" H 7150 4300 50  0000 R CNN
 F 2 "Capacitors_SMD:C_0805_HandSoldering" H 6950 4250 50  0001 C CNN
@@
 	3300 4900 3300 4850
 $Comp
-L GND #PWR017
+L GND #PWR022
 U 1 1 59C94986
 P 3600 4950
-F 0 "#PWR017" H 3600 4700 50  0001 C CNN
+F 0 "#PWR022" H 3600 4700 50  0001 C CNN
 F 1 "GND" H 3600 4800 50  0000 C CNN
 F 2 "" H 3600 4950 50  0001 C CNN
