File: controller.sch (KiCad schematic (older format))
At the start: 21 parts, among them J2 UART, J3 programming header, J4 Micro_SD_Card_Det, SW2 RAM~FLASH, SW3 start, SW4 stop, SW5 Rotary_Encoder_Switch, U1 WM8778-units, U5 STM32F401RC, U6 lcd, Y1 CSTLS4M00G53-B0

Commit message: ksch: move SDdetect pin to PA15 to make routing easier
Connections:
- wire segments 60 -> 73
Changed lines of the file:
@@
 $EndComp
 Wire Wire Line
-	7650 1550 7800 1550
+	7650 1550 7750 1550
+Wire Wire Line
+	7750 1550 7800 1550
 $Comp
 L STM32F401RC U5
@@
 $EndComp
 Wire Wire Line
-	6700 2700 7800 2700
+	6700 2700 7200 2700
+Wire Wire Line
+	7200 2700 7800 2700
 $Comp
 L STM32F401RC U5
@@
 	7200 2150 7800 2150
 Wire Wire Line
-	6700 2800 7800 2800
-Wire Wire Line
-	6700 2900 7800 2900
+	6700 2800 7250 2800
+Wire Wire Line
+	7250 2800 7800 2800
+Wire Wire Line
+	6700 2900 7300 2900
+Wire Wire Line
+	7300 2900 7800 2900
 Wire Wire Line
 	7250 2800 7250 2250
@@
 Connection ~ 7750 1550
 Wire Wire Line
-	6700 1800 7800 1800
-Wire Wire Line
-	6700 1900 7800 1900
+	6700 1800 7150 1800
+Wire Wire Line
+	7150 1800 7800 1800
+Wire Wire Line
+	6700 1900 6850 1900
+Wire Wire Line
+	6850 1900 7800 1900
 Text Label 6700 1800 2    60   ~ 0
 I2C1_SDA
@@
 Connection ~ 7150 1800
 Wire Wire Line
-	6850 1550 7300 1550
+	6850 1550 7150 1550
+Wire Wire Line
+	7150 1550 7300 1550
 Connection ~ 7150 1550
 Text Label 7300 1550 0    60   ~ 0
@@
 $EndComp
 Wire Wire Line
-	6700 4650 7400 4650
+	6700 4650 6800 4650
+Wire Wire Line
+	6800 4650 7400 4650
 $Comp
 L R_Small R4
@@
 Text Label 6700 4650 2    60   ~ 0
 SDdetect
-Text Label 3300 5550 0    60   ~ 0
+Text Label 3300 700  0    60   ~ 0
 SDdetect
 Text Label 7400 4450 2    60   ~ 0
@@
 $EndComp
 Wire Wire Line
-	8650 5700 8900 5700
+	8650 5700 8700 5700
+Wire Wire Line
+	8700 5700 8900 5700
 Wire Wire Line
 	8050 5700 7850 5700
@@
 $EndComp
 Wire Wire Line
-	8650 5500 9150 5500
+	8650 5500 8900 5500
+Wire Wire Line
+	8900 5500 9150 5500
 Text Label 8900 5300 0    60   ~ 0
 3.3V
@@
 3.3V
 Wire Wire Line
-	8000 6200 8200 6200
+	8000 6200 8100 6200
+Wire Wire Line
+	8100 6200 8200 6200
 $Comp
 L GND #PWR029
@@
 	5150 2650 5150 3000
 Wire Wire Line
-	5150 3000 5250 3000
+	5150 3000 5200 3000
+Wire Wire Line
+	5200 3000 5250 3000
 $Comp
 L GND #PWR024
@@
 $EndComp
 Wire Wire Line
-	5250 3950 5250 4400
+	5250 3950 5250 4300
+Wire Wire Line
+	5250 4300 5250 4400
 Connection ~ 5250 4300
 $Comp

Commit message: ksch: move stomp buttons to make routing easier
Connections:
- wire segments 73 -> 60
Changed lines of the file:
@@
 $EndComp
 Wire Wire Line
-	7650 1550 7750 1550
-Wire Wire Line
-	7750 1550 7800 1550
+	7650 1550 7800 1550
 $Comp
 L STM32F401RC U5
@@
 $EndComp
 Wire Wire Line
-	6700 2700 7200 2700
-Wire Wire Line
-	7200 2700 7800 2700
+	6700 2700 7800 2700
 $Comp
 L STM32F401RC U5
@@
 	7200 2150 7800 2150
 Wire Wire Line
-	6700 2800 7250 2800
-Wire Wire Line
-	7250 2800 7800 2800
-Wire Wire Line
-	6700 2900 7300 2900
-Wire Wire Line
-	7300 2900 7800 2900
+	6700 2800 7800 2800
+Wire Wire Line
+	6700 2900 7800 2900
 Wire Wire Line
 	7250 2800 7250 2250
@@
 Connection ~ 7750 1550
 Wire Wire Line
-	6700 1800 7150 1800
-Wire Wire Line
-	7150 1800 7800 1800
-Wire Wire Line
-	6700 1900 6850 1900
-Wire Wire Line
-	6850 1900 7800 1900
+	6700 1800 7800 1800
+Wire Wire Line
+	6700 1900 7800 1900
 Text Label 6700 1800 2    60   ~ 0
 I2C1_SDA
@@
 Connection ~ 7150 1800
 Wire Wire Line
-	6850 1550 7150 1550
-Wire Wire Line
-	7150 1550 7300 1550
+	6850 1550 7300 1550
 Connection ~ 7150 1550
 Text Label 7300 1550 0    60   ~ 0
@@
 $EndComp
 Wire Wire Line
-	6700 4650 6800 4650
-Wire Wire Line
-	6800 4650 7400 4650
+	6700 4650 7400 4650
 $Comp
 L R_Small R4
@@
 $EndComp
 Wire Wire Line
-	8650 5700 8700 5700
-Wire Wire Line
-	8700 5700 8900 5700
+	8650 5700 8900 5700
 Wire Wire Line
 	8050 5700 7850 5700
@@
 $EndComp
 Wire Wire Line
-	8650 5500 8900 5500
-Wire Wire Line
-	8900 5500 9150 5500
+	8650 5500 9150 5500
 Text Label 8900 5300 0    60   ~ 0
 3.3V
@@
 3.3V
 Wire Wire Line
-	8000 6200 8100 6200
-Wire Wire Line
-	8100 6200 8200 6200
+	8000 6200 8200 6200
 $Comp
 L GND #PWR029
@@
 	5150 2650 5150 3000
 Wire Wire Line
-	5150 3000 5200 3000
-Wire Wire Line
-	5200 3000 5250 3000
+	5150 3000 5250 3000
 $Comp
 L GND #PWR024
@@
 $EndComp
 Wire Wire Line
-	5250 3950 5250 4300
-Wire Wire Line
-	5250 4300 5250 4400
+	5250 3950 5250 4400
 Connection ~ 5250 4300
 $Comp
@@
 Text Label 4850 4300 2    60   ~ 0
 stomp_stop
-Text Label 1800 1450 2    60   ~ 0
+Text Label 3300 1750 0    60   ~ 0
 stomp_start
-Text Label 1800 1750 2    60   ~ 0
+Text Label 3300 1450 0    60   ~ 0
 stomp_stop
 Text Label 3300 2250 0    60   ~ 0
